Commit message: commit code

File: transbot_base/transbot_description/urdf/transbot_normal_for_autorace_2020.urdf.xacro (robot description, xacro)
@@ -31,5 +31,5 @@
     </inertial>
   </link>
-  <joint name="wheel_left_joint" type="continuous">
+  <joint name="wheel_left_rear_joint" type="continuous">
     <parent link="base_link"/>
     <child link="wheel_left_link"/>
@@ -59,5 +59,5 @@
       </inertial>
   </link>
-  <joint name="wheel_right_joint" type="continuous">
+  <joint name="wheel_right_rear_joint" type="continuous">
     <parent link="base_link"/>
     <child link="wheel_right_link"/>
@@ -86,4 +86,20 @@
                izz="2.0712558e-03" />
       </inertial>
+  </link>
+<joint name="wheel_left_front_joint" type="continuous">
+    <parent link="base_link"/>
+    <child link="wheel_left_front_link"/>
+    <origin xyz="0.0 0.1105 0.01625" rpy="-1.57 0 0"/>
+    <axis xyz="0 0 1"/>
+  </joint>
+  <link name="wheel_left_front_link">
+  </link>
+  <joint name="wheel_right_front_joint" type="continuous">
+    <parent link="base_link"/>
+    <child link="wheel_right_front_link"/>
+    <origin xyz="0.0 -0.1105 0.01625" rpy="-1.57 0 0"/>
+    <axis xyz="0 0 1"/>
+  </joint>
+  <link name="wheel_right_front_link">
   </link>
   <joint name="caster_back_joint" type="fixed">
