Commit message: commit code

File: transbot_base/transbot_description/urdf/transbot_mecanum.urdf.xacro (robot description, xacro)
@@ -1,6 +1,6 @@
 <?xml version="1.0" ?>
-<robot name="transbot_normal_for_autorace" xmlns:xacro="http://ros.org/wiki/xacro">
+<robot name="transbot_normal" xmlns:xacro="http://ros.org/wiki/xacro">
   <xacro:include filename="$(find transbot_description)/urdf/common_properties.xacro"/>
-  <xacro:include filename="$(find transbot_description)/urdf/transbot_normal_for_autorace.gazebo.xacro"/>
+  <xacro:include filename="$(find transbot_description)/urdf/transbot_normal.gazebo.xacro"/>
   <link name="base_footprint"/>
   <joint name="base_joint" type="fixed">
@@ -41,5 +41,5 @@
       <origin xyz="0 0 0" rpy="1.57 0 0"/>
       <geometry>
-        <mesh filename="package://transbot_description/meshes/wheels/left_normal.stl" scale="0.001 0.001 0.001"/>
+        <mesh filename="package://transbot_description/meshes/wheels/left_mecanum_rear.stl" scale="0.001 0.001 0.001"/>
       </geometry>
       <material name="dark"/>
@@ -69,23 +69,23 @@
       <origin xyz="0 0 0" rpy="1.57 0 0"/>
       <geometry>
-        <mesh filename="package://transbot_description/meshes/wheels/right_normal.stl" scale="0.001 0.001 0.001"/>
-      </geometry>
-      <material name="dark"/>
-    </visual>
-    <collision>
-      <origin xyz="0 0 0" rpy="0 0 0"/>
-      <geometry>
-        <cylinder length="0.018" radius="0.033"/>
-      </geometry>
-    </collision>
-    <inertial>
-      <origin xyz="0 0 0" />
-      <mass value="2.8498940e-02" />
-      <inertia ixx="1.1175580e-05" ixy="-4.2369783e-11" ixz="-5.9381719e-09"
-               iyy="1.1192413e-05" iyz="-1.4400107e-11"
-               izz="2.0712558e-05" />
-      </inertial>
-  </link>
-<joint name="wheel_left_front_joint" type="continuous">
+        <mesh filename="package://transbot_description/meshes/wheels/right_mecanum_rear.stl" scale="0.001 0.001 0.001"/>
+      </geometry>
+      <material name="dark"/>
+    </visual>
+    <collision>
+      <origin xyz="0 0 0" rpy="0 0 0"/>
+      <geometry>
+        <cylinder length="0.018" radius="0.033"/>
+      </geometry>
+    </collision>
+    <inertial>
+      <origin xyz="0 0 0" />
+      <mass value="2.8498940e-02" />
+      <inertia ixx="1.1175580e-05" ixy="-4.2369783e-11" ixz="-5.9381719e-09"
+               iyy="1.1192413e-05" iyz="-1.4400107e-11"
+               izz="2.0712558e-05" />
+      </inertial>
+  </link>
+ <joint name="wheel_left_front_joint" type="continuous">
     <parent link="base_link"/>
     <child link="wheel_left_front_link"/>
@@ -94,4 +94,24 @@
   </joint>
   <link name="wheel_left_front_link">
+    <visual>
+      <origin xyz="0 0 0" rpy="1.57 0 0"/>
+      <geometry>
+        <mesh filename="package://transbot_description/meshes/wheels/left_mecanum_front.stl" scale="0.001 0.001 0.001"/>
+      </geometry>
+      <material name="dark"/>
+    </visual>
+    <collision>
+      <origin xyz="0 0 0" rpy="0 0 0"/>
+      <geometry>
+        <cylinder length="0.018" radius="0.033"/>
+      </geometry>
+    </collision>
+    <inertial>
+      <origin xyz="0 0 0" />
+      <mass value="2.8498940e-02" />
+      <inertia ixx="1.1175580e-05" ixy="-4.2369783e-11" ixz="-5.9381719e-09"
+               iyy="1.1192413e-05" iyz="-1.4400107e-11"
+               izz="2.0712558e-05" />
+      </inertial>
   </link>
   <joint name="wheel_right_front_joint" type="continuous">
@@ -102,4 +122,24 @@
   </joint>
   <link name="wheel_right_front_link">
+    <visual>
+      <origin xyz="0 0 0" rpy="1.57 0 0"/>
+      <geometry>
+        <mesh filename="package://transbot_description/meshes/wheels/right_mecanum_front.stl" scale="0.001 0.001 0.001"/>
+      </geometry>
+      <material name="dark"/>
+    </visual>
+    <collision>
+      <origin xyz="0 0 0" rpy="0 0 0"/>
+      <geometry>
+        <cylinder length="0.018" radius="0.033"/>
+      </geometry>
+    </collision>
+    <inertial>
+      <origin xyz="0 0 0" />
+      <mass value="2.8498940e-02" />
+      <inertia ixx="1.1175580e-05" ixy="-4.2369783e-11" ixz="-5.9381719e-09"
+               iyy="1.1192413e-05" iyz="-1.4400107e-11"
+               izz="2.0712558e-05" />
+      </inertial>
   </link>
   <joint name="caster_back_joint" type="fixed">
@@ -117,5 +157,5 @@
     <inertial>
       <origin xyz="0 0 0" />
-      <mass value="0.005" />
+      <mass value="0.05" />
       <inertia ixx="0.001" ixy="0.0" ixz="0.0"
                iyy="0.001" iyz="0.0"
@@ -129,5 +169,5 @@
   </joint>
   <link name="imu_link"/>
- <joint name="scan_joint" type="fixed">
+  <joint name="scan_joint" type="fixed">
     <parent link="base_link"/>
     <child link="base_scan"/>

File: transbot_base/transbot_description/urdf/transbot_normal.urdf.xacro (robot description, xacro)
@@ -7,9 +7,9 @@
     <parent link="base_footprint"/>
     <child link="base_link"/>
-    <origin xyz="0.0 0.0 0.010" rpy="0 0 0"/>
+    <origin xyz="0.0 0.0 0.015" rpy="0 0 0"/>
   </joint>
   <link name="base_link">
     <visual>
-      <origin xyz="-0.04575 0 0.0" rpy="0 0 0"/>
+      <origin xyz="-0.053 0 0.0" rpy="0 0 0"/>
       <geometry>
         <mesh filename="package://transbot_description/meshes/bases/normal_base.stl" scale="0.001 0.001 0.001"/>
@@ -34,5 +34,5 @@
     <parent link="base_link"/>
     <child link="wheel_left_link"/>
-    <origin xyz="0.0 0.1105 0.01625" rpy="-1.57 0 0"/>
+    <origin xyz="0.0 0.1155 0.01625" rpy="-1.57 0 0"/>
     <axis xyz="0 0 1"/>
   </joint>
@@ -62,5 +62,5 @@
     <parent link="base_link"/>
     <child link="wheel_right_link"/>
-    <origin xyz="0.0 -0.1105 0.01625" rpy="-1.57 0 0"/>
+    <origin xyz="0.0 -0.1155 0.01625" rpy="-1.57 0 0"/>
     <axis xyz="0 0 1"/>
   </joint>
@@ -90,5 +90,5 @@
     <parent link="base_link"/>
     <child link="wheel_left_front_link"/>
-    <origin xyz="0.0 0.1105 0.01625" rpy="-1.57 0 0"/>
+    <origin xyz="-0.0915 0.1155 0.01625" rpy="-1.57 0 0"/>
     <axis xyz="0 0 1"/>
   </joint>
@@ -98,5 +98,5 @@
     <parent link="base_link"/>
     <child link="wheel_right_front_link"/>
-    <origin xyz="0.0 -0.1105 0.01625" rpy="-1.57 0 0"/>
+    <origin xyz="-0.0915 -0.1155 0.01625" rpy="-1.57 0 0"/>
     <axis xyz="0 0 1"/>
   </joint>
@@ -132,5 +132,5 @@
     <parent link="base_link"/>
     <child link="base_scan"/>
-    <origin xyz="0.0 0 0.184" rpy="0 0 0"/>
+    <origin xyz="0.0 0 0.192" rpy="0 0 0"/>
   </joint>
   <link name="base_scan">
@@ -157,5 +157,5 @@
   </link>
  <joint name="camera_joint" type="fixed">
-    <origin xyz="0.040 -0.011 0.130" rpy="0 0.174 0"/>
+    <origin xyz="0.0332 0.0 0.0934" rpy="0 0 0"/>
     <parent link="base_link"/>
     <child link="camera_link"/>
@@ -163,5 +163,5 @@
   <link name="camera_link">
     <collision>
-      <origin xyz="0.005 0.011 0.013" rpy="0 0 0"/>
+      <origin xyz="0.0 0.0 0.0" rpy="0 0 0"/>
       <geometry>
         <box size="0.015 0.030 0.027"/>
@@ -170,5 +170,5 @@
   </link>
   <joint name="camera_rgb_joint" type="fixed">
-    <origin xyz="0.003 0.011 0.009" rpy="0 0 0"/>
+    <origin xyz="0.0 0.0 0.0" rpy="0 0 0"/>
     <parent link="camera_link"/>
     <child link="camera_rgb_frame"/>

File: transbot_base/transbot_description/urdf/transbot_normal_for_autorace_2020.urdf.xacro (robot description, xacro)
@@ -7,9 +7,9 @@
     <parent link="base_footprint"/>
     <child link="base_link"/>
-    <origin xyz="0.0 0.0 0.010" rpy="0 0 0"/>
+    <origin xyz="0.0 0.0 0.015" rpy="0 0 0"/>
   </joint>
   <link name="base_link">
     <visual>
-      <origin xyz="-0.04575 0 0.0" rpy="0 0 0"/>
+      <origin xyz="-0.053 0 0.0" rpy="0 0 0"/>
       <geometry>
         <mesh filename="package://transbot_description/meshes/bases/normal_base.stl" scale="0.001 0.001 0.001"/>
@@ -34,12 +34,12 @@
     <parent link="base_link"/>
     <child link="wheel_left_link"/>
-    <origin xyz="0.0 0.08 0.023" rpy="-1.5707 0 0"/>
+    <origin xyz="0.0 0.1155 0.01625" rpy="-1.57 0 0"/>
     <axis xyz="0 0 1"/>
   </joint>
   <link name="wheel_left_link">
     <visual>
-      <origin xyz="0 0 0" rpy="1.5707 0 0"/>
+      <origin xyz="0 0 0" rpy="1.57 0 0"/>
       <geometry>
-        <mesh filename="package://transbot_description/meshes/wheels/left_tire.stl" scale="0.001 0.001 0.001"/>
+        <mesh filename="package://transbot_description/meshes/wheels/left_normal.stl" scale="0.001 0.001 0.001"/>
       </geometry>
       <material name="dark"/>
@@ -53,8 +53,8 @@
     <inertial>
       <origin xyz="0 0 0" />
-      <mass value="2.8498940" />
-      <inertia ixx="1.1175580e-03" ixy="-4.2369783e-08" ixz="-5.9381719e-07"
-               iyy="1.1192413e-03" iyz="-1.4400107e-08"
-               izz="2.0712558e-03" />
+      <mass value="2.8498940e-02" />
+      <inertia ixx="1.1175580e-05" ixy="-4.2369783e-11" ixz="-5.9381719e-09"
+               iyy="1.1192413e-05" iyz="-1.4400107e-11"
+               izz="2.0712558e-05" />
       </inertial>
   </link>
@@ -62,12 +62,12 @@
     <parent link="base_link"/>
     <child link="wheel_right_link"/>
-    <origin xyz="0.0 -0.080 0.023" rpy="-1.5707 0 0"/>
+    <origin xyz="0.0 -0.1155 0.01625" rpy="-1.57 0 0"/>
     <axis xyz="0 0 1"/>
   </joint>
   <link name="wheel_right_link">
     <visual>
-      <origin xyz="0 0 0" rpy="1.5707 0 0"/>
+      <origin xyz="0 0 0" rpy="1.57 0 0"/>
       <geometry>
-        <mesh filename="package://transbot_description/meshes/wheels/right_tire.stl" scale="0.001 0.001 0.001"/>
+        <mesh filename="package://transbot_description/meshes/wheels/right_normal.stl" scale="0.001 0.001 0.001"/>
       </geometry>
       <material name="dark"/>
@@ -81,8 +81,8 @@
     <inertial>
       <origin xyz="0 0 0" />
-      <mass value="2.8498940" />
-      <inertia ixx="1.1175580e-03" ixy="-4.2369783e-08" ixz="-5.9381719e-07"
-               iyy="1.1192413e-03" iyz="-1.4400107e-08"
-               izz="2.0712558e-03" />
+      <mass value="2.8498940e-02" />
+      <inertia ixx="1.1175580e-05" ixy="-4.2369783e-11" ixz="-5.9381719e-09"
+               iyy="1.1192413e-05" iyz="-1.4400107e-11"
+               izz="2.0712558e-05" />
       </inertial>
   </link>
@@ -90,5 +90,5 @@
     <parent link="base_link"/>
     <child link="wheel_left_front_link"/>
-    <origin xyz="0.0 0.1105 0.01625" rpy="-1.57 0 0"/>
+    <origin xyz="-0.0915 0.1155 0.01625" rpy="-1.57 0 0"/>
     <axis xyz="0 0 1"/>
   </joint>
@@ -98,5 +98,5 @@
     <parent link="base_link"/>
     <child link="wheel_right_front_link"/>
-    <origin xyz="0.0 -0.1105 0.01625" rpy="-1.57 0 0"/>
+    <origin xyz="-0.0915 -0.1155 0.01625" rpy="-1.57 0 0"/>
     <axis xyz="0 0 1"/>
   </joint>
@@ -129,8 +129,8 @@
   </joint>
   <link name="imu_link"/>
-  <joint name="scan_joint" type="fixed">
+ <joint name="scan_joint" type="fixed">
     <parent link="base_link"/>
     <child link="base_scan"/>
-    <origin xyz="0.0 0 0.1925" rpy="0 0 0"/>
+    <origin xyz="0.0 0 0.192" rpy="0 0 0"/>
   </joint>
   <link name="base_scan">
@@ -138,5 +138,5 @@
       <origin xyz="0 0 0.0" rpy="0 0 0"/>
       <geometry>
-        <mesh filename="package://transbot_description/meshes/sensors/yd-g4.stl" scale="0.001 0.001 0.001"/>
+        <mesh filename="package://transbot_description/meshes/sensors/yd-x2l.stl" scale="0.001 0.001 0.001"/>
       </geometry>
       <material name="dark"/>
@@ -157,5 +157,5 @@
   </link>
   <joint name="camera_dummy_joint" type="fixed">
-    <origin xyz="0.03465 0 0.09339" rpy="0 0 0"/>
+    <origin xyz="0.0332 0.0 0.0934" rpy="0 0 0"/>
     <parent link="base_link"/>
     <child link="camera_dummy_link"/>
@@ -163,5 +163,5 @@
   <link name="camera_dummy_link">
     <collision>
-      <origin xyz="0.005 0.000 0.013" rpy="0 0 0"/>
+      <origin xyz="0.0 0.0 0.0" rpy="0 0 0"/>
       <geometry>
         <box size="0.015 0.030 0.027"/>
@@ -170,5 +170,5 @@
   </link>
   <joint name="camera_joint" type="fixed">
-    <origin xyz="0.0446 0.000 0.000" rpy="0 0 0"/>
+    <origin xyz="0.0 0.0 0.0" rpy="0 0 0"/>
     <parent link="camera_dummy_link"/>
     <child link="camera_frame"/>

File: transbot_base/transbot_description/urdf/transbot_onmi.urdf.xacro (robot description, xacro)
@@ -1,6 +1,6 @@
 <?xml version="1.0" ?>
-<robot name="transbot_normal_for_autorace" xmlns:xacro="http://ros.org/wiki/xacro">
+<robot name="transbot_normal" xmlns:xacro="http://ros.org/wiki/xacro">
   <xacro:include filename="$(find transbot_description)/urdf/common_properties.xacro"/>
-  <xacro:include filename="$(find transbot_description)/urdf/transbot_normal_for_autorace.gazebo.xacro"/>
+  <xacro:include filename="$(find transbot_description)/urdf/transbot_normal.gazebo.xacro"/>
   <link name="base_footprint"/>
   <joint name="base_joint" type="fixed">
@@ -34,5 +34,5 @@
     <parent link="base_link"/>
     <child link="wheel_left_link"/>
-    <origin xyz="0.0 0.1155 0.01625" rpy="-1.57 0 0"/>
+    <origin xyz="0.0442 0.0975 0.01625" rpy="-1.57 0 -0.785"/>
     <axis xyz="0 0 1"/>
   </joint>
@@ -41,5 +41,5 @@
       <origin xyz="0 0 0" rpy="1.57 0 0"/>
       <geometry>
-        <mesh filename="package://transbot_description/meshes/wheels/left_normal.stl" scale="0.001 0.001 0.001"/>
+        <mesh filename="package://transbot_description/meshes/wheels/onmi.stl" scale="0.001 0.001 0.001"/>
       </geometry>
       <material name="dark"/>
@@ -62,5 +62,5 @@
     <parent link="base_link"/>
     <child link="wheel_right_link"/>
-    <origin xyz="0.0 -0.1155 0.01625" rpy="-1.57 0 0"/>
+    <origin xyz="0.0442 -0.0975 0.01625" rpy="-1.57 0 0.785"/>
     <axis xyz="0 0 1"/>
   </joint>
@@ -69,37 +69,77 @@
       <origin xyz="0 0 0" rpy="1.57 0 0"/>
       <geometry>
-        <mesh filename="package://transbot_description/meshes/wheels/right_normal.stl" scale="0.001 0.001 0.001"/>
-      </geometry>
-      <material name="dark"/>
-    </visual>
-    <collision>
-      <origin xyz="0 0 0" rpy="0 0 0"/>
-      <geometry>
-        <cylinder length="0.018" radius="0.033"/>
-      </geometry>
-    </collision>
-    <inertial>
-      <origin xyz="0 0 0" />
-      <mass value="2.8498940e-02" />
-      <inertia ixx="1.1175580e-05" ixy="-4.2369783e-11" ixz="-5.9381719e-09"
-               iyy="1.1192413e-05" iyz="-1.4400107e-11"
-               izz="2.0712558e-05" />
-      </inertial>
-  </link>
-<joint name="wheel_left_front_joint" type="continuous">
+        <mesh filename="package://transbot_description/meshes/wheels/onmi.stl" scale="0.001 0.001 0.001"/>
+      </geometry>
+      <material name="dark"/>
+    </visual>
+    <collision>
+      <origin xyz="0 0 0" rpy="0 0 0"/>
+      <geometry>
+        <cylinder length="0.018" radius="0.033"/>
+      </geometry>
+    </collision>
+    <inertial>
+      <origin xyz="0 0 0" />
+      <mass value="2.8498940e-02" />
+      <inertia ixx="1.1175580e-05" ixy="-4.2369783e-11" ixz="-5.9381719e-09"
+               iyy="1.1192413e-05" iyz="-1.4400107e-11"
+               izz="2.0712558e-05" />
+      </inertial>
+  </link>
+ <joint name="wheel_left_front_joint" type="continuous">
     <parent link="base_link"/>
     <child link="wheel_left_front_link"/>
-    <origin xyz="-0.0915 0.1155 0.01625" rpy="-1.57 0 0"/>
+    <origin xyz="-0.1505 0.0975 0.01625" rpy="-1.57 0 0.785"/>
     <axis xyz="0 0 1"/>
   </joint>
   <link name="wheel_left_front_link">
+    <visual>
+      <origin xyz="0 0 0" rpy="1.57 0 0"/>
+      <geometry>
+        <mesh filename="package://transbot_description/meshes/wheels/onmi.stl" scale="0.001 0.001 0.001"/>
+      </geometry>
+      <material name="dark"/>
+    </visual>
+    <collision>
+      <origin xyz="0 0 0" rpy="0 0 0"/>
+      <geometry>
+        <cylinder length="0.018" radius="0.033"/>
+      </geometry>
+    </collision>
+    <inertial>
+      <origin xyz="0 0 0" />
+      <mass value="2.8498940e-02" />
+      <inertia ixx="1.1175580e-05" ixy="-4.2369783e-11" ixz="-5.9381719e-09"
+               iyy="1.1192413e-05" iyz="-1.4400107e-11"
+               izz="2.0712558e-05" />
+      </inertial>
   </link>
   <joint name="wheel_right_front_joint" type="continuous">
     <parent link="base_link"/>
     <child link="wheel_right_front_link"/>
-    <origin xyz="-0.0915 -0.1155 0.01625" rpy="-1.57 0 0"/>
+    <origin xyz="-0.1505 -0.0975 0.01625" rpy="-1.57 0 -0.785"/>
     <axis xyz="0 0 1"/>
   </joint>
   <link name="wheel_right_front_link">
+    <visual>
+      <origin xyz="0 0 0" rpy="1.57 0 0"/>
+      <geometry>
+        <mesh filename="package://transbot_description/meshes/wheels/onmi.stl" scale="0.001 0.001 0.001"/>
+      </geometry>
+      <material name="dark"/>
+    </visual>
+    <collision>
+      <origin xyz="0 0 0" rpy="0 0 0"/>
+      <geometry>
+        <cylinder length="0.018" radius="0.033"/>
+      </geometry>
+    </collision>
+    <inertial>
+      <origin xyz="0 0 0" />
+      <mass value="2.8498940e-02" />
+      <inertia ixx="1.1175580e-05" ixy="-4.2369783e-11" ixz="-5.9381719e-09"
+               iyy="1.1192413e-05" iyz="-1.4400107e-11"
+               izz="2.0712558e-05" />
+      </inertial>
   </link>
   <joint name="caster_back_joint" type="fixed">
@@ -117,5 +157,5 @@
     <inertial>
       <origin xyz="0 0 0" />
-      <mass value="0.005" />
+      <mass value="0.05" />
       <inertia ixx="0.001" ixy="0.0" ixz="0.0"
                iyy="0.001" iyz="0.0"
@@ -129,5 +169,5 @@
   </joint>
   <link name="imu_link"/>
- <joint name="scan_joint" type="fixed">
+  <joint name="scan_joint" type="fixed">
     <parent link="base_link"/>
     <child link="base_scan"/>

Commit message: commit code

File: transbot_base/transbot_description/urdf/transbot_mecanum.urdf.xacro (robot description, xacro)
@@ -11,5 +11,5 @@
   <link name="base_link">
     <visual>
-      <origin xyz="-0.053 0 0.0" rpy="0 0 0"/>
+      <origin xyz="-0.04575 0 0.0" rpy="0 0 0"/>
       <geometry>
         <mesh filename="package://transbot_description/meshes/bases/normal_base.stl" scale="0.001 0.001 0.001"/>

File: transbot_base/transbot_description/urdf/transbot_normal.urdf.xacro (robot description, xacro)
@@ -11,5 +11,5 @@
   <link name="base_link">
     <visual>
-      <origin xyz="-0.053 0 0.0" rpy="0 0 0"/>
+      <origin xyz="-0.04575 0 0.0" rpy="0 0 0"/>
       <geometry>
         <mesh filename="package://transbot_description/meshes/bases/normal_base.stl" scale="0.001 0.001 0.001"/>

File: transbot_base/transbot_description/urdf/transbot_onmi.urdf.xacro (robot description, xacro)
@@ -11,5 +11,5 @@
   <link name="base_link">
     <visual>
-      <origin xyz="-0.053 0 0.0" rpy="0 0 0"/>
+      <origin xyz="-0.04575 0 0.0" rpy="0 0 0"/>
       <geometry>
         <mesh filename="package://transbot_description/meshes/bases/normal_base.stl" scale="0.001 0.001 0.001"/>
