Commit message: commit code

File: transbot_base/transbot_description/urdf/miniarm.urdf.xacro (robot description, xacro)
@@ -32,5 +32,5 @@
     <parent link="link1"/>
     <child link="link2"/>
-    <origin xyz="0.012 0.0 0.017" rpy="0 0 0"/>
+    <origin xyz="0.0 0.0 0.017" rpy="0 0 0"/>
     <axis xyz="0 0 1"/>
     <limit velocity="4.8" effort="1" lower="${-pi*0.9}" upper="${pi*0.9}" />
@@ -39,5 +39,5 @@
   <link name="link2">
     <visual>
-      <origin xyz="0 0 0.018" rpy="0 0 0"/>
+      <origin xyz="0 0 0.0207" rpy="0 0 0"/>
       <geometry>
         <mesh filename="package://transbot_description/meshes/arm/chain_link2.stl" scale="0.001 0.001 0.001"/>
@@ -46,5 +46,5 @@
     </visual>
     <collision>
-      <origin xyz="0 0 0.018" rpy="0 0 0"/>
+      <origin xyz="0 0 0.0207" rpy="0 0 0"/>
       <geometry>
         <mesh filename="package://transbot_description/meshes/arm/chain_link2.stl" scale="0.001 0.001 0.001"/>
@@ -63,5 +63,5 @@
     <parent link="link2"/>
     <child link="link3"/>
-    <origin xyz="0.0 0.0 0.058" rpy="0 0 0"/>
+    <origin xyz="0.0 0.0 0.060" rpy="0 0 0"/>
     <axis xyz="0 1 0"/>
     <limit velocity="4.8" effort="1" lower="${-pi*0.57}" upper="${pi*0.5}" />
@@ -125,5 +125,5 @@
     <parent link="link4"/>
     <child link="link5"/>
-    <origin xyz="0.124 0.0 0.0" rpy="0 0 0"/>
+    <origin xyz="0.129 0.0 0.0" rpy="0 0 0"/>
     <axis xyz="0 1 0"/>
     <limit velocity="4.8" effort="1" lower="${-pi*0.57}" upper="${pi*0.65}" />
@@ -183,5 +183,5 @@
     <parent link="link5"/>
     <child link="gripper_link"/>
-    <origin xyz="0.0817 0.021 0.0" rpy="0 0 0"/>
+    <origin xyz="0.098 0.021 0.0" rpy="0 0 0"/>
     <axis xyz="0 1 0"/>
     <limit velocity="4.8" effort="1" lower="-0.010" upper="0.019" />
@@ -214,5 +214,5 @@
     <parent link="link5"/>
     <child link="gripper_link_sub"/>
-    <origin xyz="0.0817 -0.021 0" rpy="0 0 0"/>
+    <origin xyz="0.098 -0.021 0" rpy="0 0 0"/>
     <axis xyz="0 -1 0"/>
     <limit velocity="4.8" effort="1" lower="-0.010" upper="0.019" />
