Commit message: fix simulation problem

File: transbot_base/transbot_description/urdf/transbot_normal.gazebo.xacro (robot description, xacro)
@@ -3,4 +3,5 @@
   <xacro:arg name="laser_visual" default="false"/>
   <xacro:arg name="imu_visual"   default="false"/>
+  <xacro:arg name="camera_visual" default="false"/>
   <gazebo reference="base_link">
     <material>Gazebo/DarkGrey</material>
@@ -124,3 +125,36 @@
     </sensor>
   </gazebo>
+ <!--link : https://www.raspberrypi.org/documentation/hardware/camera/-->
+  <gazebo reference="camera_rgb_frame">
+    <sensor type="camera" name="Pi Camera">
+      <always_on>true</always_on>
+      <visualize>$(arg camera_visual)</visualize>
+      <camera>
+          <horizontal_fov>1.085595</horizontal_fov>
+          <image>
+              <width>320</width>
+              <height>240</height>
+              <format>R8G8B8</format>
+          </image>
+          <clip>
+              <near>0.03</near>
+              <far>100</far>
+          </clip>
+      </camera>
+      <plugin name="camera_controller" filename="libgazebo_ros_camera.so">
+        <alwaysOn>true</alwaysOn>
+        <updateRate>30.0</updateRate>
+        <cameraName>camera</cameraName>
+        <frameName>camera_rgb_optical_frame</frameName>
+        <imageTopicName>image</imageTopicName>
+        <cameraInfoTopicName>camera_info</cameraInfoTopicName>
+        <hackBaseline>0.07</hackBaseline>
+        <distortionK1>0.0</distortionK1>
+        <distortionK2>0.0</distortionK2>
+        <distortionK3>0.0</distortionK3>
+        <distortionT1>0.0</distortionT1>
+        <distortionT2>0.0</distortionT2>
+      </plugin>
+    </sensor>
+  </gazebo>
 </robot>

File: transbot_base/transbot_description/urdf/transbot_normal.urdf.xacro (robot description, xacro)
@@ -140,3 +140,28 @@
     </inertial>
   </link>
+ <joint name="camera_joint" type="fixed">
+    <origin xyz="0.040 -0.011 0.130" rpy="0 0.174 0"/>
+    <parent link="base_link"/>
+    <child link="camera_link"/>
+  </joint>
+  <link name="camera_link">
+    <collision>
+      <origin xyz="0.005 0.011 0.013" rpy="0 0 0"/>
+      <geometry>
+        <box size="0.015 0.030 0.027"/>
+      </geometry>
+    </collision>
+  </link>
+  <joint name="camera_rgb_joint" type="fixed">
+    <origin xyz="0.003 0.011 0.009" rpy="0 0 0"/>
+    <parent link="camera_link"/>
+    <child link="camera_rgb_frame"/>
+  </joint>
+  <link name="camera_rgb_frame"/>
+  <joint name="camera_rgb_optical_joint" type="fixed">
+    <origin xyz="0 0 0" rpy="-1.57 0 -1.57"/>
+    <parent link="camera_rgb_frame"/>
+    <child link="camera_rgb_optical_frame"/>
+  </joint>
+  <link name="camera_rgb_optical_frame"/>
 </robot>

Commit message: 修改为使用X2激光雷达、修改urdf中的支撑轮质量

File: transbot_base/transbot_description/urdf/transbot_normal.gazebo.xacro (robot description, xacro)
@@ -102,5 +102,5 @@
         <scan>
           <horizontal>
-            <samples>24</samples>
+            <samples>360</samples>
             <resolution>1</resolution>
             <min_angle>0.0</min_angle>

File: transbot_base/transbot_description/urdf/transbot_normal.urdf.xacro (robot description, xacro)
@@ -101,5 +101,5 @@
     <inertial>
       <origin xyz="0 0 0" />
-      <mass value="0.005" />
+      <mass value="0.05" />
       <inertia ixx="0.001" ixy="0.0" ixz="0.0"
                iyy="0.001" iyz="0.0"

Commit message: fix urdf problem

File: transbot_base/transbot_description/urdf/transbot_normal.gazebo.xacro (robot description, xacro)
@@ -56,7 +56,7 @@
       <legacyMode>false</legacyMode>
       <updateRate>30</updateRate>
-      <leftJoint>wheel_left_joint</leftJoint>
-      <rightJoint>wheel_right_joint</rightJoint>
-      <wheelSeparation>0.221</wheelSeparation>
+      <leftJoint>wheel_left_rear_joint</leftJoint>
+      <rightJoint>wheel_right_rear_joint</rightJoint>
+      <wheelSeparation>0.231</wheelSeparation>
       <wheelDiameter>0.066</wheelDiameter>
       <wheelAcceleration>1</wheelAcceleration>

File: transbot_base/transbot_description/urdf/transbot_normal.urdf.xacro (robot description, xacro)
@@ -87,5 +87,5 @@
       </inertial>
   </link>
-<joint name="wheel_left_front_joint" type="continuous">
+<joint name="wheel_left_front_joint" type="fixed">
     <parent link="base_link"/>
     <child link="wheel_left_front_link"/>
@@ -95,5 +95,5 @@
   <link name="wheel_left_front_link">
   </link>
-  <joint name="wheel_right_front_joint" type="continuous">
+  <joint name="wheel_right_front_joint" type="fixed">
     <parent link="base_link"/>
     <child link="wheel_right_front_link"/>
