Commit message: change

File: transbot_base/transbot_description/urdf/transbot_normal.urdf.xacro (robot description, xacro)
@@ -31,5 +31,5 @@
     </inertial>
   </link>
-  <joint name="wheel_left_joint" type="continuous">
+  <joint name="wheel_left_rear_joint" type="continuous">
     <parent link="base_link"/>
     <child link="wheel_left_link"/>
@@ -59,5 +59,5 @@
       </inertial>
   </link>
-  <joint name="wheel_right_joint" type="continuous">
+  <joint name="wheel_right_rear_joint" type="continuous">
     <parent link="base_link"/>
     <child link="wheel_right_link"/>

Commit message: commit code

File: transbot_base/transbot_description/urdf/transbot_normal.urdf.xacro (robot description, xacro)
@@ -87,4 +87,20 @@
       </inertial>
   </link>
+<joint name="wheel_left_front_joint" type="continuous">
+    <parent link="base_link"/>
+    <child link="wheel_left_front_link"/>
+    <origin xyz="0.0 0.1105 0.01625" rpy="-1.57 0 0"/>
+    <axis xyz="0 0 1"/>
+  </joint>
+  <link name="wheel_left_front_link">
+  </link>
+  <joint name="wheel_right_front_joint" type="continuous">
+    <parent link="base_link"/>
+    <child link="wheel_right_front_link"/>
+    <origin xyz="0.0 -0.1105 0.01625" rpy="-1.57 0 0"/>
+    <axis xyz="0 0 1"/>
+  </joint>
+  <link name="wheel_right_front_link">
+  </link>
   <joint name="caster_back_joint" type="fixed">
     <parent link="base_link"/>

Commit message: commit code

File: transbot_base/transbot_description/urdf/transbot_normal.urdf.xacro (robot description, xacro)
@@ -41,5 +41,5 @@
       <origin xyz="0 0 0" rpy="1.57 0 0"/>
       <geometry>
-        <mesh filename="package://transbot_description/meshes/wheels/left_tire.stl" scale="0.001 0.001 0.001"/>
+        <mesh filename="package://transbot_description/meshes/wheels/left_normal.stl" scale="0.001 0.001 0.001"/>
       </geometry>
       <material name="dark"/>
@@ -69,5 +69,5 @@
       <origin xyz="0 0 0" rpy="1.57 0 0"/>
       <geometry>
-        <mesh filename="package://transbot_description/meshes/wheels/right_tire.stl" scale="0.001 0.001 0.001"/>
+        <mesh filename="package://transbot_description/meshes/wheels/right_normal.stl" scale="0.001 0.001 0.001"/>
       </geometry>
       <material name="dark"/>
@@ -132,5 +132,5 @@
     <parent link="base_link"/>
     <child link="base_scan"/>
-    <origin xyz="0.0 0 0.1925" rpy="0 0 0"/>
+    <origin xyz="0.0 0 0.184" rpy="0 0 0"/>
   </joint>
   <link name="base_scan">
@@ -138,5 +138,5 @@
       <origin xyz="0 0 0.0" rpy="0 0 0"/>
       <geometry>
-        <mesh filename="package://transbot_description/meshes/sensors/yd-g4.stl" scale="0.001 0.001 0.001"/>
+        <mesh filename="package://transbot_description/meshes/sensors/yd-x2l.stl" scale="0.001 0.001 0.001"/>
       </geometry>
       <material name="dark"/>

File: transbot_base/transbot_description/urdf/transbot_normal_for_autorace.urdf.xacro (robot description, xacro)
@@ -41,5 +41,5 @@
       <origin xyz="0 0 0" rpy="1.57 0 0"/>
       <geometry>
-        <mesh filename="package://transbot_description/meshes/wheels/left_tire.stl" scale="0.001 0.001 0.001"/>
+        <mesh filename="package://transbot_description/meshes/wheels/left_rear.stl" scale="0.001 0.001 0.001"/>
       </geometry>
       <material name="dark"/>
@@ -69,5 +69,5 @@
       <origin xyz="0 0 0" rpy="1.57 0 0"/>
       <geometry>
-        <mesh filename="package://transbot_description/meshes/wheels/right_tire.stl" scale="0.001 0.001 0.001"/>
+        <mesh filename="package://transbot_description/meshes/wheels/right_rear.stl" scale="0.001 0.001 0.001"/>
       </geometry>
       <material name="dark"/>

Commit message: commit code

File: transbot_base/transbot_description/urdf/transbot_normal.urdf.xacro (robot description, xacro)
@@ -87,5 +87,5 @@
       </inertial>
   </link>
-<joint name="wheel_left_front_joint" type="fixed">
+<joint name="wheel_left_front_joint" type="continuous">
     <parent link="base_link"/>
     <child link="wheel_left_front_link"/>
@@ -95,5 +95,5 @@
   <link name="wheel_left_front_link">
   </link>
-  <joint name="wheel_right_front_joint" type="fixed">
+  <joint name="wheel_right_front_joint" type="continuous">
     <parent link="base_link"/>
     <child link="wheel_right_front_link"/>

File: transbot_base/transbot_description/urdf/transbot_normal_miniarm.urdf.xacro (robot description, xacro)
@@ -1,5 +1,5 @@
 <?xml version="1.0"?>
 <robot name="transbot_miniarm" xmlns:xacro="http://ros.org/wiki/xacro">
-  <!-- Include Transbot Waffle URDF -->
+  <!-- Include Transbot URDF -->
   <xacro:include filename="$(find transbot_description)/urdf/transbot_normal.urdf.xacro"/>
   <!-- Include MINIARM URDF -->
